Commit message: Working on Talos URDF

File: robotcontrollerclient/resources/meshes/talos.urdf (robot description, URDF)
Before this commit: robot talos, 15 links, 14 joints
Links:
- link Arm: geometry collision mesh filename=TalosArm.stl scale=1 1 1; visual mesh filename=TalosArm.stl scale=1 1 1
- link Bucket: geometry collision box size=0.40 0.30 0.18; visual mesh filename=TalosBucket.stl scale=1 1 1
Joints:
- joint Arm_Joint: origin xyz=0.180193 -0.033254 0.283140 rpy=0 0 0 -> xyz=0 0 0 rpy=0 0 0
- joint Bucket_Joint: origin xyz=0.741492 -0.00775 -0.320993 rpy=0 0 0 -> xyz=0 0 0 rpy=0 0 0

Commit message: Fixed Talos

File: robotcontrollerclient/resources/meshes/talos.urdf (robot description, URDF)
Before this commit: robot talos, 15 links, 14 joints
Links:
- removed link Camera_Mount
Joints:
- removed joint Camera_Mount_Joint
- joint Arm_Joint: origin xyz=0 0 0 rpy=0 0 0 -> xyz=-0.319 0.18 0.171 rpy=0.0304533 0 0
- joint BL_Wheel_Joint: origin xyz=0.18387 0 0.23588 rpy=0 0 0 -> xyz=-0.3315 0.28 0.089 rpy=0 0 0
- joint BR_Wheel_Joint: origin xyz=0.183875 -0.475667 0.235883 rpy=0 0 -3.14159 -> xyz=-0.3315 -0.20 0.089 rpy=0 0 -3.14159
- joint Bucket_Joint: origin xyz=0 0 0 rpy=0 0 0 -> xyz=0.913 -0.020 -0.079 rpy=0 0 0
- joint FL_Wheel_Joint: origin xyz=0.8411 -0.019814 0.235883 rpy=0 0 0 -> xyz=0.3275 0.265 0.089 rpy=0 0 0
- joint FR_Wheel_Joint: origin xyz=0.8411 -0.538167 0.235883 rpy=0 0 0 -> xyz=0.3275 -0.27 0.089 rpy=0 0 0
- joint base_to_zed2i: origin xyz=0.822000 0.083000 0.508000 rpy=0 0 0 -> xyz=0.3275 -0.27 0.35 rpy=0 0 0

Commit message: Working on URDF

File: robotcontrollerclient/resources/meshes/talos.urdf (robot description, URDF)
Before this commit: robot talos, 14 links, 13 joints
Joints:
- joint Arm_Joint: limit lower=-0.7 upper=0.3 effort=120 velocity=1.5 -> lower=-0.7 upper=0.0873 effort=120 velocity=1.5
- joint Bucket_Joint: limit lower=-0.45 upper=1.25 effort=80 velocity=2.0 -> lower=-0.45 upper=2.2 effort=80 velocity=2.0
